Commit message: Changes der Verzweiflung

File: src/ur10e_moveit_config/config/simple_table.urdf.xacro (robot description, xacro)
@@ -14,13 +14,12 @@
       <collision>
         <geometry>
-          <box size="1.2 0.8 0.05"/>
+          <box size="5.0 5.0 0.05"/>
         </geometry>
       </collision>
       <inertial>
-        <mass value="5.0"/>
-        <inertia ixx="0.1" ixy="0.0" ixz="0.0"
-                 iyy="0.1" iyz="0.0"
-                 izz="0.1"/>
-        <origin xyz="0 0 0" rpy="0 0 0"/>
+        <mass value="10000.0"/> <origin xyz="0 0 0" rpy="0 0 0"/>
+        <inertia ixx="208333.3" ixy="0.0" ixz="0.0"
+                 iyy="208333.3" iyz="0.0"
+                 izz="416666.7"/>
       </inertial>
     </link>

File: src/ur10e_moveit_config/config/ur10e_robot.urdf.xacro (robot description, xacro)
@@ -17,5 +17,5 @@
         <child link="base_link"/>
         <!-- Z-Versatz entspricht Tischhöhe (0.05 m dick) -->
-        <origin xyz="0 0 0.10" rpy="0 0 0"/>
+        <origin xyz="0 0 0.025" rpy="0 0 0"/>
     </joint>
     <!-- ROS2 control plugin -->
