Commit message: Fehlerhafte Version, ohne richtige controller

File: install/ur10e_moveit_config/share/ur10e_moveit_config/config/simple_table.urdf.xacro (robot description, xacro)
@@ -1 +1,32 @@
-/home/matteo-melzer/ws_moveit/src/ur10e_moveit_config/config/simple_table.urdf.xacro
+<?xml version="1.0"?>
+<robot xmlns:xacro="http://ros.org/wiki/xacro">
+  <!-- Macro-Definition für einen simplen Tisch -->
+  <xacro:macro name="simple_table" params="prefix parent xyz:='0 0 0' rpy:='0 0 0'">
+    <link name="${prefix}table_top">
+      <visual>
+        <geometry>
+          <box size="5.0 5.0 0.05"/> <!-- Länge, Breite, Höhe -->
+        </geometry>
+        <material name="brown">
+          <color rgba="0.6 0.4 0.2 1"/>
+        </material>
+      </visual>
+      <collision>
+        <geometry>
+          <box size="5.0 5.0 0.05"/>
+        </geometry>
+      </collision>
+      <inertial>
+        <mass value="10000.0"/> <origin xyz="0 0 0" rpy="0 0 0"/>
+        <inertia ixx="208333.3" ixy="0.0" ixz="0.0"
+                 iyy="208333.3" iyz="0.0"
+                 izz="416666.7"/>
+      </inertial>
+    </link>
+    <joint name="${prefix}table_fixed" type="fixed">
+      <parent link="${parent}"/>
+      <child link="${prefix}table_top"/>
+      <origin xyz="${xyz}" rpy="${rpy}"/>
+    </joint>
+  </xacro:macro>
+</robot>

File: install/ur10e_moveit_config/share/ur10e_moveit_config/config/ur10e_robot.ros2_control.xacro (robot description, xacro)
@@ -1 +1,58 @@
-/home/matteo-melzer/ws_moveit/src/ur10e_moveit_config/config/ur10e_robot.ros2_control.xacro
+<?xml version="1.0"?>
+<robot xmlns:xacro="http://www.ros.org/wiki/xacro">
+    <xacro:macro name="ur10e_robot_ros2_control" params="controllers_file initial_positions_file">
+        <xacro:property name="initial_positions" value="${xacro.load_yaml(initial_positions_file)}"/>
+        <ros2_control name="GazeboSystem" type="system">
+            <hardware>
+                <plugin>gazebo_ros2_control/GazeboSystem</plugin>
+            </hardware>
+            <joint name="shoulder_pan_joint">
+                <command_interface name="position"/>
+                <state_interface name="position">
+                    <param name="initial_value">${initial_positions['shoulder_pan_joint']}</param>
+                </state_interface>
+                <state_interface name="velocity"/>
+            </joint>
+            <joint name="shoulder_lift_joint">
+                <command_interface name="position"/>
+                <state_interface name="position">
+                    <param name="initial_value">${initial_positions['shoulder_lift_joint']}</param>
+                </state_interface>
+                <state_interface name="velocity"/>
+            </joint>
+            <joint name="elbow_joint">
+                <command_interface name="position"/>
+                <state_interface name="position">
+                    <param name="initial_value">${initial_positions['elbow_joint']}</param>
+                </state_interface>
+                <state_interface name="velocity"/>
+            </joint>
+            <joint name="wrist_1_joint">
+                <command_interface name="position"/>
+                <state_interface name="position">
+                    <param name="initial_value">${initial_positions['wrist_1_joint']}</param>
+                </state_interface>
+                <state_interface name="velocity"/>
+            </joint>
+            <joint name="wrist_2_joint">
+                <command_interface name="position"/>
+                <state_interface name="position">
+                    <param name="initial_value">${initial_positions['wrist_2_joint']}</param>
+                </state_interface>
+                <state_interface name="velocity"/>
+            </joint>
+            <joint name="wrist_3_joint">
+                <command_interface name="position"/>
+                <state_interface name="position">
+                    <param name="initial_value">${initial_positions['wrist_3_joint']}</param>
+                </state_interface>
+                <state_interface name="velocity"/>
+            </joint>
+        </ros2_control>
+        <gazebo>
+            <plugin name="gazebo_ros2_control" filename="libgazebo_ros2_control.so">
+                <parameters>${controllers_file}</parameters>
+            </plugin>
+        </gazebo>
+    </xacro:macro>
+</robot>

File: install/ur10e_moveit_config/share/ur10e_moveit_config/config/ur10e_robot.urdf.xacro (robot description, xacro)
@@ -1 +1,19 @@
-/home/matteo-melzer/ws_moveit/src/ur10e_moveit_config/config/ur10e_robot.urdf.xacro
+<?xml version="1.0"?>
+<robot xmlns:xacro="http://www.ros.org/wiki/xacro" name="ur10e_robot">
+    <xacro:arg name="controllers_file" default="ros2_controllers.yaml"/>
+    <xacro:arg name="initial_positions_file" default="initial_positions.yaml"/>
+    <link name="world"/>
+    <xacro:include filename="$(find ur_description)/urdf/ur10e.urdf" />
+    <xacro:include filename="ur10e_robot.ros2_control.xacro" />
+    <xacro:include filename="$(find ur10e_moveit_config)/config/simple_table.urdf.xacro"/>
+    <xacro:simple_table prefix="table_" parent="world" xyz="0 0 0" rpy="0 0 0"/>
+    <joint name="ur10e_on_table" type="fixed">
+        <parent link="table_table_top"/>
+        <child link="base_link"/>
+        <origin xyz="0 0 0.025" rpy="0 0 0"/>
+    </joint>
+    <xacro:ur10e_robot_ros2_control
+        controllers_file="$(arg controllers_file)"
+        initial_positions_file="$(arg initial_positions_file)"
+    />
+</robot>

File: src/ur10e_moveit_config/config/ur10e_robot.ros2_control.xacro (robot description, xacro)
@@ -1,15 +1,14 @@
 <?xml version="1.0"?>
 <robot xmlns:xacro="http://www.ros.org/wiki/xacro">
-    <xacro:macro name="ur10e_robot_ros2_control" params="name initial_positions_file">
-        <xacro:property name="initial_positions" value="${load_yaml(initial_positions_file)['initial_positions']}"/>
-        <ros2_control name="${name}" type="system">
+    <xacro:macro name="ur10e_robot_ros2_control" params="controllers_file initial_positions_file">
+        <xacro:property name="initial_positions" value="${xacro.load_yaml(initial_positions_file)}"/>
+        <ros2_control name="GazeboSystem" type="system">
             <hardware>
-                <!-- By default, set up controllers for simulation. This won't work on real hardware -->
-                <plugin>mock_components/GenericSystem</plugin>
+                <plugin>gazebo_ros2_control/GazeboSystem</plugin>
             </hardware>
             <joint name="shoulder_pan_joint">
                 <command_interface name="position"/>
                 <state_interface name="position">
-                  <param name="initial_value">${initial_positions['shoulder_pan_joint']}</param>
+                    <param name="initial_value">${initial_positions['shoulder_pan_joint']}</param>
                 </state_interface>
                 <state_interface name="velocity"/>
@@ -18,5 +17,5 @@
                 <command_interface name="position"/>
                 <state_interface name="position">
-                  <param name="initial_value">${initial_positions['shoulder_lift_joint']}</param>
+                    <param name="initial_value">${initial_positions['shoulder_lift_joint']}</param>
                 </state_interface>
                 <state_interface name="velocity"/>
@@ -25,5 +24,5 @@
                 <command_interface name="position"/>
                 <state_interface name="position">
-                  <param name="initial_value">${initial_positions['elbow_joint']}</param>
+                    <param name="initial_value">${initial_positions['elbow_joint']}</param>
                 </state_interface>
                 <state_interface name="velocity"/>
@@ -32,5 +31,5 @@
                 <command_interface name="position"/>
                 <state_interface name="position">
-                  <param name="initial_value">${initial_positions['wrist_1_joint']}</param>
+                    <param name="initial_value">${initial_positions['wrist_1_joint']}</param>
                 </state_interface>
                 <state_interface name="velocity"/>
@@ -39,5 +38,5 @@
                 <command_interface name="position"/>
                 <state_interface name="position">
-                  <param name="initial_value">${initial_positions['wrist_2_joint']}</param>
+                    <param name="initial_value">${initial_positions['wrist_2_joint']}</param>
                 </state_interface>
                 <state_interface name="velocity"/>
@@ -46,9 +45,14 @@
                 <command_interface name="position"/>
                 <state_interface name="position">
-                  <param name="initial_value">${initial_positions['wrist_3_joint']}</param>
+                    <param name="initial_value">${initial_positions['wrist_3_joint']}</param>
                 </state_interface>
                 <state_interface name="velocity"/>
             </joint>
         </ros2_control>
+        <gazebo>
+            <plugin name="gazebo_ros2_control" filename="libgazebo_ros2_control.so">
+                <parameters>${controllers_file}</parameters>
+            </plugin>
+        </gazebo>
     </xacro:macro>
 </robot>

File: src/ur10e_moveit_config/config/ur10e_robot.urdf.xacro (robot description, xacro)
@@ -1,30 +1,19 @@
 <?xml version="1.0"?>
 <robot xmlns:xacro="http://www.ros.org/wiki/xacro" name="ur10e_robot">
-    <xacro:arg name="initial_positions_file" default="initial_positions.yaml" />
-    <!-- Dummy link "world" als Basis der Szene -->
+    <xacro:arg name="controllers_file" default="ros2_controllers.yaml"/>
+    <xacro:arg name="initial_positions_file" default="initial_positions.yaml"/>
     <link name="world"/>
-    <!-- Import ur10e_robot URDF -->
     <xacro:include filename="$(find ur_description)/urdf/ur10e.urdf" />
-    <!-- Import ros2_control -->
     <xacro:include filename="ur10e_robot.ros2_control.xacro" />
-    <!-- Import table macro -->
     <xacro:include filename="$(find ur10e_moveit_config)/config/simple_table.urdf.xacro"/>
-    <!-- Instantiate table and attach to world -->
     <xacro:simple_table prefix="table_" parent="world" xyz="0 0 0" rpy="0 0 0"/>
-    <!-- Fix the UR10e base on top of the table -->
     <joint name="ur10e_on_table" type="fixed">
         <parent link="table_table_top"/>
         <child link="base_link"/>
-        <!-- Z-Versatz entspricht Tischhöhe (0.05 m dick) -->
         <origin xyz="0 0 0.025" rpy="0 0 0"/>
     </joint>
-    <!-- ROS2 control plugin -->
-    <xacro:ur10e_robot_ros2_control name="GazeboSystem" initial_positions_file="$(arg initial_positions_file)"/>
-    <!-- ros2_control Gazebo Plugin -->
-    <gazebo>
-    <plugin name="gazebo_ros2_control" filename="libgazebo_ros2_control.so">
-        <robot_namespace>/</robot_namespace>
-        <ros_control_namespace>/</ros_control_namespace>
-    </plugin>
-    </gazebo>
+    <xacro:ur10e_robot_ros2_control
+        controllers_file="$(arg controllers_file)"
+        initial_positions_file="$(arg initial_positions_file)"
+    />
 </robot>
